Commit message: feat: add payload to parkour URDF

File: source/instinctlab/instinctlab/tasks/parkour/urdf/g1_29dof_torsoBase_popsicle_with_shoe.urdf (robot description, URDF)
Before this commit: robot g1, 40 links, 39 joints
Links:
- added link payload_link, mass 1.34; collision mesh filename=meshes/payload_link.STL; visual mesh filename=meshes/payload_link.STL
Joints:
- added joint payload_joint: type fixed, parent torso_link, child payload_link, origin xyz=-0.062 0 0.055 rpy=0 0 0

Commit message: fix(parkour URDF): Increase cylinder lengths in collision geometry
Update cylinder lengths by 0.02 in both left and right foot collision geometry
sections to improve collision detection accuracy.

File: source/instinctlab/instinctlab/tasks/parkour/urdf/g1_29dof_torsoBase_popsicle_with_shoe.urdf (robot description, URDF)
Before this commit: robot g1, 40 links, 39 joints
Links:
- link left_ankle_roll_link: geometry collision cylinder length=0.07 radius=0.01; collision cylinder length=0.07 radius=0.01
- link right_ankle_roll_link: geometry collision cylinder length=0.07 radius=0.01; collision cylinder length=0.07 radius=0.01
