Commit message: robot: use BeyondMimic main.urdf (pelvis root); rebuild shoe variant; align base heights
- robot URDF content replaced with whole_body_tracking unitree_description
  main.urdf (pelvis floating base); mesh paths adapted to in-repo assets
- G1_29DOF_TORSOBASE_POPSICLE_CFG init pos 0.82 -> 0.76
- parkour: init pos/target_height 0.9 -> 0.76, root_height termination 0.5 -> 0.36
- dcm_planner: z0 0.82 -> 0.76 (base height in normal standing posture)
- parkour shoe URDF rebuilt on top of main.urdf (foot sole 23mm lower)

File: source/instinctlab/instinctlab/assets/resources/unitree_g1/urdf/g1_29dof_torsobase_popsicle.urdf (robot description, URDF)
Before this commit: robot g1, 40 links, 39 joints
Joints:
- joint waist_pitch_joint: child waist_roll_link -> torso_link; parent torso_link -> waist_roll_link
- joint waist_roll_joint: child waist_yaw_link -> waist_roll_link; origin xyz=0.0039635 0 -0.044 rpy=0 0 0 -> xyz=-0.0039635 0 0.044 rpy=0 0 0; parent waist_roll_link -> waist_yaw_link
- joint waist_yaw_joint: child pelvis -> waist_yaw_link; parent waist_yaw_link -> pelvis

File: source/instinctlab/instinctlab/tasks/parkour/urdf/g1_29dof_torsoBase_popsicle_with_shoe.urdf (robot description, URDF)
Before this commit: robot g1, 40 links, 39 joints
Joints:
- joint waist_pitch_joint: child waist_roll_link -> torso_link; parent torso_link -> waist_roll_link
- joint waist_roll_joint: child waist_yaw_link -> waist_roll_link; origin xyz=0.0039635 0 -0.044 rpy=0 0 0 -> xyz=-0.0039635 0 0.044 rpy=0 0 0; parent waist_roll_link -> waist_yaw_link
- joint waist_yaw_joint: child pelvis -> waist_yaw_link; parent waist_yaw_link -> pelvis
